File: 216/we_need_to_talk/we_need_to_talk_schematic/we_need_to_talk_schematic.kicad_sch (KiCad schematic)
At the start: 0 parts

Commit message: esp schematic, still need rpi
Parts:
- added 1: ESP32-NODEMCU-S3, symbol MECPS:ESP32-NODEMCU-S3
- added D1, D2, D3, D4, D5: LED, symbol Device:LED
- added R1: R_Photo, symbol Device:R_Photo
- added R2, R3, R4, R5, R6, R7: R_US, symbol Device:R_US
Connections:
- new net: D2.1 (K), R4.1
- new net: R4.2, R5.2, R6.2, R7.2
- new net: D1.1 (K), R3.1
- new net: 1. (GND), R2.2, R3.2
- new net: 1. (GND), R1.1
- new net: 1.5 (GPIO36), R1.2, R2.1
- new net: D4.1 (K), R6.1
- new net: D5.1 (K), R7.1
- new net: 1.40 (GPIO3), D1.2 (A)
- new net: D3.1 (K), R5.1

Commit message: refactoring code
Parts:
- removed D1: LED, symbol Device:LED
- removed R3: R_US, symbol Device:R_US
- added R8: R_US, symbol Device:R_US
- added SW1: SW_Push, Button_Switch_SMD:Nidec_Copal_CAS-120A, symbol Switch:SW_Push
- added U1: (no value), Package_SO:QSOP-24_3.9x8.7mm_P0.635mm, symbol mecps:rpi_expansion
Connections:
- net at D2.2 (A): now also U1.16 (GPIO23)
- net at R4.2, R5.2, R6.2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: now also R8.2, U1.6 (GND)
- net at D4.2 (A): now also U1.22 (GPIO25)
- net at D5.2 (A): now also U1.24 (GPIO8)
- net at D3.2 (A): now also U1.18 (GPIO24)
- new net: SW1.1, U1.40 (GPIO21)
- new net: R8.1, SW1.2
Other:
- note added: "ESP32"
- note added: "Raspberry Pi"
- moved on the sheet: D2, D3, D4, D5, R1, R2, R4, R5, R6, R7
